Commit message: Modifications from Yan's catkinization.

File: kingfisher_description/urdf/base.urdf.xacro (robot description, xacro)
@@ -40,8 +40,33 @@
     xmlns:xacro="http://ros.org/wiki/xacro" name="kingfisher">
 	<!-- Included URDF/XACRO Files -->
-    <kingfisher_include filename="$(find kingfisher_description)/urdf/parts.urdf.xacro" />
+    <include filename="$(find kingfisher_description)/urdf/parts.urdf.xacro" />
     <!-- PROPERTY LIST -->
     <!--All units in m-kg-s-radians unit system -->
     <property name="M_PI" value="3.1415926535897931" />
+    <!-- BASE-FOOTPRINT -->
+    <!-- base_footprint is a fictitious link(frame) that is on the ground right below base_link origin, navigation stack depends on this frame -->
+    <link name="base_footprint">
+        <inertial>
+            <mass value="0.0001" />
+            <origin xyz="0 0 0" />
+            <inertia ixx="0.0001" ixy="0.0" ixz="0.0"
+                iyy="0.0001" iyz="0.0"
+                izz="0.0001" />
+        </inertial>
+        <visual>
+            <origin xyz="0 0 0" rpy="0 0 0" />
+            <geometry>
+                <box size="0.001 0.001 0.001" />
+            </geometry>
+        </visual>
+    </link>
+    <gazebo reference="base_footprint">
+        <turnGravityOff>false</turnGravityOff>
+    </gazebo>
+    <joint name="base_footprint_joint" type="fixed">
+		<origin xyz="0 0 0" rpy="0 0 0" />
+        <parent link="base_footprint"/>
+        <child link="base_link" />
+    </joint>
     <!-- BASE-LINK -->
     <!--Actual body/chassis of the robot-->
@@ -57,5 +82,5 @@
             <origin xyz="0 0 0" rpy="${M_PI/2} 0 ${M_PI/2}" />
             <geometry>
-                <mesh filename="package://kingfisher_description/mesh/kingfisher_base.stl" />
+                <mesh filename="package://kingfisher_description/meshes/kingfisher_base.stl" />
             </geometry>
         </visual>
@@ -73,19 +98,19 @@
     <!-- PANEL-LINKS -->
     <!-- Top Plate -->
-    <kingfisher_part parent="base_link" name="left_panel" mesh="left_panel"
+    <kingfisher_part parent="base_footprint" name="left_panel" mesh="left_panel"
           translateX="0.0" translateY="-0.35" translateZ="0.05"
           rotateX="${M_PI/2}" rotateY="0.0" rotateZ="${M_PI/2}"/>
-    <gazebo reference="base_link_left_panel_part">
+    <gazebo reference="base_footprint_left_panel_part">
         <material>Gazebo/Yellow</material>
     </gazebo>
-    <kingfisher_part parent="base_link" name="right_panel" mesh="right_panel"
+    <kingfisher_part parent="base_footprint" name="right_panel" mesh="right_panel"
           translateX="0.0" translateY="0.35" translateZ="0.05"
           rotateX="${M_PI/2}" rotateY="0.0" rotateZ="${-M_PI/2}"/>
-    <gazebo reference="base_link_right_panel_part">
+    <gazebo reference="base_footprint_right_panel_part">
         <material>Gazebo/Yellow</material>
     </gazebo>
     <!--Gazebo Plugin for simulating Kingfisher dynamics-->
     <gazebo>
-        <controller:kingfisher_plugin name="kingfisher_dynamic" plugin="libkingfisher_gazebo_plugins.so">
+	    <plugin name="kingfisher_dynamic" filename="libkingfisher_gazebo_plugins.so">
             <maxForce>62.0</maxForce>
             <bodyName>base_link</bodyName>
@@ -95,5 +120,5 @@
             <yawDampingFactor>20.0</yawDampingFactor>
             <rolPitDampingFactor>5.0</rolPitDampingFactor>
-        </controller:kingfisher_plugin>
+        </plugin>
     </gazebo>
 </robot>

File: kingfisher_description/urdf/parts.urdf.xacro (robot description, xacro)
@@ -62,5 +62,5 @@
 				<origin xyz="0 0 0" rpy="0 0 0" />
 				<geometry>
-					<mesh filename="package://kingfisher_description/mesh/${mesh}.stl" />
+					<mesh filename="package://kingfisher_description/meshes/${mesh}.stl" />
 				</geometry>
 			</visual>

File: kingfisher_description/urdf/standard.urdf.xacro (robot description, xacro)
@@ -5,22 +5,8 @@
     xmlns:interface="http://playerstage.sourceforge.net/gazebo/xmlschema/#interface">
     <!-- Included URDF Files -->
-    <kingfisher_include filename="$(find kingfisher_description)/urdf/base.urdf.xacro" />
-    <!-- Set up gps configuration -->
-    <gazebo>
-        <controller:kingfisher_gps_plugin name="kingfisher_gps" plugin="libkingfisher_ros_gps.so">
-            <alwaysOn>true</alwaysOn>
-            <updateRate>4.0</updateRate>
-            <bodyName>base_link</bodyName>
-            <topicName>fix</topicName>
-            <velocityTopicName>fix_velocity</velocityTopicName>
-            <drift>5.0 5.0 5.0</drift>
-            <gaussianNoise>0.1 0.1 0.1</gaussianNoise>
-            <velocityDrift>0 0 0</velocityDrift>
-            <velocityGaussianNoise>0.1 0.1 0.1</velocityGaussianNoise>
-        </controller:kingfisher_gps_plugin>
-    </gazebo>
+    <include filename="$(find kingfisher_description)/urdf/base.urdf.xacro" />
     <!-- Set up imu configuration -->
     <gazebo>
-        <controller:kingfisher_imu_plugin name="kingfisher_imu" plugin="libkingfisher_ros_imu.so">
+        <plugin name="kingfisher_imu" filename="libgazebo_ros_imu.so">
             <updateRate>100.0</updateRate>
             <bodyName>base_link</bodyName>
@@ -34,5 +20,5 @@
             <headingDrift>0.1</headingDrift>
             <headingGaussianNoise>0.05</headingGaussianNoise>
-        </controller:kingfisher_imu_plugin>
+        </plugin>
     </gazebo>
     <!-- Set up camera linkage and configuration -->
@@ -50,69 +36,41 @@
     </link>
     <gazebo reference="camera_link">
-        <sensor:camera name="camera_sensor">
-            <imageSize>640 480</imageSize>
-            <imageFormat>BAYER_BGGR8</imageFormat>
-            <hfov>90</hfov>
-            <nearClip>0.1</nearClip>
-            <farClip>100</farClip>
-            <updateRate>25.0</updateRate>
-            <controller:gazebo_ros_camera name="camera_controller" plugin="libkingfisher_ros_prosilica.so">
+        <sensor type="camera" name="camera">
+            <update_rate>30.0</update_rate>
+            <camera name="kingfisher_camera">
+                <horizontal_fov>1.3962634</horizontal_fov>
+                <image>
+                    <width>640</width>
+                    <height>480</height>
+                    <format>R8G8B8</format>
+                </image>
+                <clip>
+                    <near>0.02</near>
+                    <far>300</far>
+                </clip>
+                <noise>
+                    <type>gaussian</type>
+                    <!-- Noise is sampled independently per pixel on each frame.
+                       That pixel's noise value is added to each of its color
+                       channels, which at that point lie in the range [0,1]. -->
+                    <mean>0.0</mean>
+                    <stddev>0.007</stddev>
+                </noise>
+            </camera>
+            <plugin name="camera_controller" filename="libgazebo_ros_camera.so">
                 <alwaysOn>true</alwaysOn>
-                <updateRate>25.0</updateRate>
-                <cameraName>camera</cameraName>
+                <updateRate>30.0</updateRate>
+                <cameraName>kingfisher/camera</cameraName>
                 <imageTopicName>image_raw</imageTopicName>
                 <cameraInfoTopicName>camera_info</cameraInfoTopicName>
                 <frameName>camera_link</frameName>
-                <CxPrime>320.5</CxPrime>
-                <Cx>320.5</Cx>
-                <Cy>240.5</Cy>
-                <!-- image_width / (2*tan(hfov_radian /2)) -->
-                <!-- 320 for wide and 772.55 for narrow stereo camera -->
-                <focal_length>320</focal_length>
-                <distortion_k1>0.0</distortion_k1>
-                <distortion_k2>0.0</distortion_k2>
-                <distortion_k3>0.0</distortion_k3>
-                <distortion_t1>0.0</distortion_t1>
-                <distortion_t2>0.0</distortion_t2>
-            </controller:gazebo_ros_camera>
-        </sensor:camera>
-        <material>Gazebo/Blue</material>
-    </gazebo>
-    <!-- Set up sonar linkage and configuration -->
-    <joint name="base_link_sonar_link_joint" type="fixed">
-		<origin xyz="0 0 -0.2" rpy="0 1.57 0" />
-        <parent link="base_link"/>
-        <child link="sonar_link" />
-    </joint>
-    <link name="sonar_link">
-        <inertial>
-            <mass value="1"/>
-            <origin xyz="0 0 0"/>
-            <inertia ixx="0.1" ixy="0.0" ixz="0.0" iyy="0.1" iyz="0.0" izz="0.1"/>
-        </inertial>
-    </link>
-    <gazebo reference="sonar_link">
-      <sensor:ray name="sonar_sensor">
-        <rayCount>5</rayCount>
-        <rangeCount>5</rangeCount>
-        <verticalRayCount>5</verticalRayCount>
-        <verticalRangeCount>5</verticalRangeCount>
-        <minAngle>-${5/2}</minAngle>
-        <verticalMinAngle>-${5/2}</verticalMinAngle>
-        <maxAngle>${5/2}</maxAngle>
-        <verticalMaxAngle>${5/2}</verticalMaxAngle>
-        <minRange>0</minRange>
-        <maxRange>30</maxRange>
-        <resRange>0.01</resRange>
-        <updateRate>20</updateRate>
-        <controller:hector_gazebo_ros_sonar name="gazebo_ros_sonar_controller" plugin="libkingfisher_ros_sonar.so">
-            <gaussianNoise>0.005</gaussianNoise>
-            <topicName>sonar</topicName>
-            <frameId>sonar_link</frameId>
-            <offset>0</offset>
-            <drift>0</drift>
-            <driftFrequency>0</driftFrequency>
-        </controller:hector_gazebo_ros_sonar>
-      </sensor:ray>
+                <hackBaseline>0.07</hackBaseline>
+                <distortionK1>0.0</distortionK1>
+                <distortionK2>0.0</distortionK2>
+                <distortionK3>0.0</distortionK3>
+                <distortionT1>0.0</distortionT1>
+                <distortionT2>0.0</distortionT2>
+            </plugin>
+        </sensor>
     </gazebo>
 </robot>

Commit message: Fix model colours, retab base file.

File: kingfisher_description/urdf/base.urdf.xacro (robot description, xacro)
@@ -39,6 +39,7 @@
     xmlns:physics="http://playerstage.sourceforge.net/gazebo/xmlschema/#physics"
     xmlns:xacro="http://ros.org/wiki/xacro" name="kingfisher">
-	<!-- Included URDF/XACRO Files -->
-    <include filename="$(find kingfisher_description)/urdf/parts.urdf.xacro" />
+    <!-- Included URDF/XACRO Files -->
+    <xacro:include filename="$(find kingfisher_description)/urdf/materials.urdf.xacro" />
+    <xacro:include filename="$(find kingfisher_description)/urdf/parts.urdf.xacro" />
     <!-- PROPERTY LIST -->
     <!--All units in m-kg-s-radians unit system -->
@@ -65,5 +66,5 @@
     </gazebo>
     <joint name="base_footprint_joint" type="fixed">
-		<origin xyz="0 0 0" rpy="0 0 0" />
+    <origin xyz="0 0 0" rpy="0 0 0" />
         <parent link="base_footprint"/>
         <child link="base_link" />
@@ -84,8 +85,9 @@
                 <mesh filename="package://kingfisher_description/meshes/kingfisher_base.stl" />
             </geometry>
+            <material name="DarkGray" />
         </visual>
         <collision>
-	        <origin xyz="0 0 0" rpy="0 0 0" />
-	        <geometry>
+          <origin xyz="0 0 0" rpy="0 0 0" />
+          <geometry>
                 <box size = "0.1 0.1 0.1"/> <!--making it slightly bigger in x and z direction-->
             </geometry>
@@ -100,5 +102,6 @@
     <kingfisher_part parent="base_footprint" name="left_panel" mesh="left_panel"
           translateX="0.0" translateY="-0.35" translateZ="0.05"
-          rotateX="${M_PI/2}" rotateY="0.0" rotateZ="${M_PI/2}"/>
+          rotateX="${M_PI/2}" rotateY="0.0" rotateZ="${M_PI/2}"
+          color="Yellow" />
     <gazebo reference="base_footprint_left_panel_part">
         <material>Gazebo/Yellow</material>
@@ -106,5 +109,6 @@
     <kingfisher_part parent="base_footprint" name="right_panel" mesh="right_panel"
           translateX="0.0" translateY="0.35" translateZ="0.05"
-          rotateX="${M_PI/2}" rotateY="0.0" rotateZ="${-M_PI/2}"/>
+          rotateX="${M_PI/2}" rotateY="0.0" rotateZ="${-M_PI/2}"
+          color="Yellow" />
     <gazebo reference="base_footprint_right_panel_part">
         <material>Gazebo/Yellow</material>
@@ -112,5 +116,5 @@
     <!--Gazebo Plugin for simulating Kingfisher dynamics-->
     <gazebo>
-	    <plugin name="kingfisher_dynamic" filename="libkingfisher_gazebo_plugins.so">
+      <plugin name="kingfisher_dynamic" filename="libkingfisher_gazebo_plugins.so">
             <maxForce>62.0</maxForce>
             <bodyName>base_link</bodyName>

File: kingfisher_description/urdf/parts.urdf.xacro (robot description, xacro)
@@ -45,5 +45,5 @@
 	<property name="iyz_com_cs" value="0.00" /> <!-- at center of mass aligned with coordinate system, kg*m^2-->
 	<property name="izz_com_cs" value="0.01" /> <!-- at center of mass aligned with coordinate system, kg*m^2-->
-	<xacro:macro name="kingfisher_part" params="parent name mesh translateX translateY translateZ rotateX rotateY rotateZ">
+	<xacro:macro name="kingfisher_part" params="parent name mesh translateX translateY translateZ rotateX rotateY rotateZ color">
 		<joint name="${parent}_${name}_joint" type="fixed">
 		    <origin xyz="${translateX} ${translateY} ${translateZ}"
@@ -64,4 +64,5 @@
 					<mesh filename="package://kingfisher_description/meshes/${mesh}.stl" />
 				</geometry>
+        <material name="${color}" />
 			</visual>
 			<collision>

File: kingfisher_description/urdf/standard.urdf.xacro (robot description, xacro)
@@ -3,7 +3,8 @@
     xmlns:sensor="http://playerstage.sourceforge.net/gazebo/xmlschema/#sensor"
     xmlns:controller="http://playerstage.sourceforge.net/gazebo/xmlschema/#controller"
-    xmlns:interface="http://playerstage.sourceforge.net/gazebo/xmlschema/#interface">
+    xmlns:interface="http://playerstage.sourceforge.net/gazebo/xmlschema/#interface"
+    xmlns:xacro="http://ros.org/wiki/xacro">
     <!-- Included URDF Files -->
-    <include filename="$(find kingfisher_description)/urdf/base.urdf.xacro" />
+    <xacro:include filename="$(find kingfisher_description)/urdf/base.urdf.xacro" />
     <!-- Set up imu configuration -->
     <gazebo>
