Commit message: Heron rename.

File: heron_description/urdf/base.urdf.xacro (robot description, xacro)
@@ -23,5 +23,5 @@
 (INCLUDING NEGLIGENCE OR OTHERWISE) ARISING IN ANY WAY OUT OF THE USE OF THIS
 SOFTWARE, EVEN IF ADVISED OF THE POSSIBILITY OF SUCH DAMAGE.
-This program contains the description of the robot base model for the Clearpath Kingfisher
+This program contains the description of the robot base model for the Clearpath Heron
 -->
 <robot
@@ -38,8 +38,8 @@
     xmlns:renderable="http://playerstage.sourceforge.net/gazebo/xmlschema/#renderable"
     xmlns:physics="http://playerstage.sourceforge.net/gazebo/xmlschema/#physics"
-    xmlns:xacro="http://ros.org/wiki/xacro" name="kingfisher">
+    xmlns:xacro="http://ros.org/wiki/xacro" name="heron">
     <!-- Included URDF/XACRO Files -->
-    <xacro:include filename="$(find kingfisher_description)/urdf/materials.urdf.xacro" />
-    <xacro:include filename="$(find kingfisher_description)/urdf/parts.urdf.xacro" />
+    <xacro:include filename="$(find heron_description)/urdf/materials.urdf.xacro" />
+    <xacro:include filename="$(find heron_description)/urdf/parts.urdf.xacro" />
     <!-- PROPERTY LIST -->
     <!--All units in m-kg-s-radians unit system -->
@@ -83,5 +83,5 @@
             <origin xyz="0 0 0" rpy="${M_PI/2} 0 ${M_PI/2}" />
             <geometry>
-                <mesh filename="package://kingfisher_description/meshes/kingfisher_base.stl" />
+                <mesh filename="package://heron_description/meshes/heron_base.stl" />
             </geometry>
             <material name="DarkGray" />
@@ -100,5 +100,5 @@
     <!-- PANEL-LINKS -->
     <!-- Top Plate -->
-    <kingfisher_part parent="base_footprint" name="left_panel" mesh="left_panel"
+    <heron_part parent="base_footprint" name="left_panel" mesh="left_panel"
           translateX="0.0" translateY="-0.35" translateZ="0.05"
           rotateX="${M_PI/2}" rotateY="0.0" rotateZ="${M_PI/2}"
@@ -107,5 +107,5 @@
         <material>Gazebo/Yellow</material>
     </gazebo>
-    <kingfisher_part parent="base_footprint" name="right_panel" mesh="right_panel"
+    <heron_part parent="base_footprint" name="right_panel" mesh="right_panel"
           translateX="0.0" translateY="0.35" translateZ="0.05"
           rotateX="${M_PI/2}" rotateY="0.0" rotateZ="${-M_PI/2}"
@@ -114,7 +114,7 @@
         <material>Gazebo/Yellow</material>
     </gazebo>
-    <!--Gazebo Plugin for simulating Kingfisher dynamics-->
+    <!--Gazebo Plugin for simulating Heron dynamics-->
     <gazebo>
-      <plugin name="kingfisher_dynamic" filename="libkingfisher_gazebo_plugins.so">
+      <plugin name="heron_dynamic" filename="libheron_gazebo_plugins.so">
             <maxForce>62.0</maxForce>
             <bodyName>base_link</bodyName>

File: heron_description/urdf/materials.urdf.xacro (robot description, xacro)
@@ -23,5 +23,5 @@
 (INCLUDING NEGLIGENCE OR OTHERWISE) ARISING IN ANY WAY OUT OF THE USE OF THIS
 SOFTWARE, EVEN IF ADVISED OF THE POSSIBILITY OF SUCH DAMAGE.
-This program contains the materials for the Clearpath Kingfisher model.
+This program contains the materials for the Clearpath Heron model.
 -->
 <robot>

File: heron_description/urdf/parts.urdf.xacro (robot description, xacro)
@@ -23,5 +23,5 @@
 (INCLUDING NEGLIGENCE OR OTHERWISE) ARISING IN ANY WAY OUT OF THE USE OF THIS
 SOFTWARE, EVEN IF ADVISED OF THE POSSIBILITY OF SUCH DAMAGE.
-This program is a macro for adding decorative parts to the Clearpath Kingfisher M200 model.
+This program is a macro for adding decorative parts to the Clearpath Heron M200 model.
 It is assumed that such parts are fixed to others, and those other parts' inertial
 parameters account for the decorative parts. Decorative parts currently do not
@@ -31,5 +31,5 @@
 	xmlns:controller="http://playerstage.sourceforge.net/gazebo/xmlschema/#controller"
 	xmlns:interface="http://playerstage.sourceforge.net/gazebo/xmlschema/#interface"
-	xmlns:xacro="http://ros.org/wiki/xacro" name="kingfisher_part">
+	xmlns:xacro="http://ros.org/wiki/xacro" name="heron_part">
 	<property name="x_com" value="0.00000000" /> <!-- com : center of mass -->
 	<property name="y_com" value="0.00000000" /> <!-- com : center of mass -->
@@ -45,5 +45,5 @@
 	<property name="iyz_com_cs" value="0.00" /> <!-- at center of mass aligned with coordinate system, kg*m^2-->
 	<property name="izz_com_cs" value="0.01" /> <!-- at center of mass aligned with coordinate system, kg*m^2-->
-	<xacro:macro name="kingfisher_part" params="parent name mesh translateX translateY translateZ rotateX rotateY rotateZ color">
+	<xacro:macro name="heron_part" params="parent name mesh translateX translateY translateZ rotateX rotateY rotateZ color">
 		<joint name="${parent}_${name}_joint" type="fixed">
 		    <origin xyz="${translateX} ${translateY} ${translateZ}"
@@ -62,5 +62,5 @@
 				<origin xyz="0 0 0" rpy="0 0 0" />
 				<geometry>
-					<mesh filename="package://kingfisher_description/meshes/${mesh}.stl" />
+					<mesh filename="package://heron_description/meshes/${mesh}.stl" />
 				</geometry>
         <material name="${color}" />

File: heron_description/urdf/standard.urdf.xacro (robot description, xacro)
@@ -1,4 +1,4 @@
 <?xml version="1.0"?>
-<robot name="kingfisher"
+<robot name="heron"
     xmlns:sensor="http://playerstage.sourceforge.net/gazebo/xmlschema/#sensor"
     xmlns:controller="http://playerstage.sourceforge.net/gazebo/xmlschema/#controller"
@@ -6,8 +6,8 @@
     xmlns:xacro="http://ros.org/wiki/xacro">
     <!-- Included URDF Files -->
-    <xacro:include filename="$(find kingfisher_description)/urdf/base.urdf.xacro" />
+    <xacro:include filename="$(find heron_description)/urdf/base.urdf.xacro" />
     <!-- Set up imu configuration -->
     <gazebo>
-        <plugin name="kingfisher_imu" filename="libgazebo_ros_imu.so">
+        <plugin name="heron_imu" filename="libgazebo_ros_imu.so">
             <updateRate>20.0</updateRate>
             <bodyName>base_link</bodyName>
@@ -25,5 +25,5 @@
     <!-- Set up gps configuration -->
     <gazebo>
-        <plugin name="kingfisher_gps" filename="libkingfisher_ros_gps.so">
+        <plugin name="heron_gps" filename="libheron_ros_gps.so">
             <alwaysOn>true</alwaysOn>
             <updateRate>10.0</updateRate>
@@ -53,5 +53,5 @@
         <sensor type="camera" name="camera">
             <update_rate>30.0</update_rate>
-            <camera name="kingfisher_camera">
+            <camera name="heron_camera">
                 <horizontal_fov>1.3962634</horizontal_fov>
                 <image>
@@ -76,5 +76,5 @@
                 <alwaysOn>true</alwaysOn>
                 <updateRate>30.0</updateRate>
-                <cameraName>kingfisher/camera</cameraName>
+                <cameraName>heron/camera</cameraName>
                 <imageTopicName>image_raw</imageTopicName>
                 <cameraInfoTopicName>camera_info</cameraInfoTopicName>
@@ -132,5 +132,5 @@
                     </noise>
                 </ray>
-                <plugin name="kingfisher_ros_sonar_controller" filename="libkingfisher_ros_sonar.so">
+                <plugin name="heron_ros_sonar_controller" filename="libheron_ros_sonar.so">
                     <gaussianNoise>0.005</gaussianNoise>
                     <topicName>sonar</topicName>
