Commit message: Fixing namespaces to allow for empty namespace

File: heron_description/urdf/accessories.urdf.xacro (robot description, xacro)
@@ -10,5 +10,5 @@
   -->
   <xacro:macro name="rear_plate" params="type namespace">
-    <link name="${namespace}/rear_plate">
+    <link name="${namespace}rear_plate">
       <visual>
         <origin xyz="0 0 0" rpy="0 0 0" />
@@ -20,9 +20,9 @@
     </link>
     <joint name="rear_plate_joint" type="fixed">
-      <parent link="${namespace}/base_link" />
-      <child link="${namespace}/rear_plate" />
+      <parent link="${namespace}base_link" />
+      <child link="${namespace}rear_plate" />
       <origin xyz="-0.1915 0.0 0.001" />
     </joint>
-    <gazebo reference="${namespace}/rear_plate">
+    <gazebo reference="${namespace}rear_plate">
       <material>Gazebo/DarkGrey</material>
     </gazebo>
@@ -35,6 +35,6 @@
     <origin xyz="$(optenv HERON_NAVSAT_SMART6_OFFSET -0.25 0 0.08)"
             rpy="$(optenv HERON_NAVSAT_SMART6_RPY 0 0 0)" />
-      <parent link="$(arg namespace)/base_link" />
-      <child link="$(arg namespace)/$(optenv HERON_NAVSAT_SMART6_MOUNT rear)_navsat" />
+      <parent link="$(arg suffix_ns)base_link" />
+      <child link="$(arg suffix_ns)$(optenv HERON_NAVSAT_SMART6_MOUNT rear)_navsat" />
     </joint>
   </xacro:if>
@@ -49,6 +49,6 @@
       <origin xyz="$(optenv HERON_LASER_OFFSET 0.0575 0 0.0115)"
               rpy="$(optenv HERON_LASER_RPY 0 0 0)" />
-      <parent link="$(arg namespace)/rear_plate" />
-      <child link="$(arg namespace)/$(optenv HERON_LASER_MOUNT front)_laser_mount" />
+      <parent link="$(arg suffix_ns)rear_plate" />
+      <child link="$(arg suffix_ns)$(optenv HERON_LASER_MOUNT front)_laser_mount" />
     </joint>
   </xacro:if>
@@ -60,19 +60,19 @@
     <origin xyz="$(optenv HERON_AXIS_PTZ_OFFSET -0.124 0 0.078)"
             rpy="$(optenv HERON_AXIS_PTZ_RPY 0 0 0)" />
-      <parent link="$(arg namespace)/rear_plate" />
-      <child link="$(arg namespace)/$(optenv HERON_AXIS_PTZ_MOUNT axis_ptz)_camera_link" />
+      <parent link="$(arg suffix_ns)rear_plate" />
+      <child link="$(arg suffix_ns)$(optenv HERON_AXIS_PTZ_MOUNT axis_ptz)_camera_link" />
     </joint>
   </xacro:if>
   <xacro:if value="$(optenv HERON_SONAR 0)">
-    <link name="$(arg namespace)/sonar_$(optenv HERON_SONAR_MOUNT surface)" />
+    <link name="$(arg suffix_ns)sonar_$(optenv HERON_SONAR_MOUNT surface)" />
     <joint name="$(optenv HERON_SONAR_MOUNT rear)_sonar_joint" type="fixed">
     <origin xyz="$(optenv HERON_SONAR_OFFSET 0.0 0 -0.10)"
             rpy="$(optenv HERON_SONAR_RPY 0 0 0)" />
-      <parent link="$(arg namespace)/base_link" />
-      <child link="$(arg namespace)/sonar_$(optenv HERON_SONAR_MOUNT surface)" />
+      <parent link="$(arg suffix_ns)base_link" />
+      <child link="$(arg suffix_ns)sonar_$(optenv HERON_SONAR_MOUNT surface)" />
     </joint>
   </xacro:if>
   <xacro:unless value="$(optenv HERON_LASER 0)">
-    <rear_plate type="plain" namespace="$(arg namespace)" />
+    <rear_plate type="plain" namespace="$(arg suffix_ns)" />
   </xacro:unless>
 </robot>

File: heron_description/urdf/actuators.xacro (robot description, xacro)
@@ -9,9 +9,9 @@
     -->
     <!-- Right Thruster -->
-    <xacro:thruster_macro robot_namespace="$(arg namespace)" thruster_id="0">
+    <xacro:thruster_macro robot_namespace="$(arg namespace)" suffix_ns="$(arg suffix_ns)" thruster_id="0">
         <origin xyz="-0.53 -0.377654 -0.16" rpy="0 0 0" />
     </xacro:thruster_macro>
     <!-- Left Thruster -->
-    <xacro:thruster_macro robot_namespace="$(arg namespace)" thruster_id="1">
+    <xacro:thruster_macro robot_namespace="$(arg namespace)" suffix_ns="$(arg suffix_ns)" thruster_id="1">
         <origin xyz="-0.53 0.377654 -0.16" rpy="0 0 0" />
     </xacro:thruster_macro>

File: heron_description/urdf/base.xacro (robot description, xacro)
@@ -27,10 +27,10 @@
   <xacro:macro name="panel" params="namespace side location">
       <!-- location flips the panel. 1 is for the left and -1 is for the right -->
-      <joint name="${namespace}/base_${side}_joint" type="fixed">
+      <joint name="${namespace}base_${side}_joint" type="fixed">
         <origin xyz="0.0 ${location * 0.34495} 0.04959" rpy="0 0 0" />
-        <parent link="${namespace}/base_link" />
-        <child link="${namespace}/${side}_panel_link" />
+        <parent link="${namespace}base_link" />
+        <child link="${namespace}${side}_panel_link" />
       </joint>
-      <link name="${namespace}/${side}_panel_link">
+      <link name="${namespace}${side}_panel_link">
         <inertial>
           <mass value="0.1" />
@@ -47,5 +47,5 @@
         </visual>
       </link>
-      <gazebo reference="${namespace}/${side}_panel_link">
+      <gazebo reference="${namespace}${side}_panel_link">
         <material>Gazebo/Yellow</material>
       </gazebo>
@@ -54,5 +54,5 @@
   <xacro:macro name="heron_base" params="namespace *gazebo">
       <!-- Rigid body description of the base link -->
-      <link name="${namespace}/base_link">
+      <link name="${namespace}base_link">
         <!--
           Be careful to setup the coefficients for the inertial tensor,
@@ -74,5 +74,5 @@
       </link>
       <!-- Dummy Link to contain the inertial information for base_link -->
-      <link name="${namespace}/dummy_link">
+      <link name="${namespace}dummy_link">
         <inertial>
           <mass value="${mass}" />
@@ -85,8 +85,8 @@
       </link>
       <joint name="dummy_to_base" type="fixed">
-        <parent link="${namespace}/base_link" />
-        <child link="${namespace}/dummy_link" />
+        <parent link="${namespace}base_link" />
+        <child link="${namespace}dummy_link" />
       </joint>
-    <gazebo reference="${namespace}/base_link">
+    <gazebo reference="${namespace}base_link">
       <selfCollide>false</selfCollide>
       <material>Gazebo/DarkGrey</material>
@@ -99,6 +99,6 @@
     <!-- Include the sensor modules -->
     <xacro:include filename="$(find heron_description)/urdf/sensors.xacro"/>
-    <xacro:panel namespace="$(arg namespace)" side="left" location="1" />
-    <xacro:panel namespace="$(arg namespace)" side="right" location="-1" />
+    <xacro:panel namespace="$(arg suffix_ns)" side="left" location="1" />
+    <xacro:panel namespace="$(arg suffix_ns)" side="right" location="-1" />
     <xacro:include filename="$(find heron_description)/urdf/accessories.urdf.xacro" />
     <!-- Optional custom includes. -->

File: heron_description/urdf/gazebo.xacro (robot description, xacro)
@@ -11,5 +11,5 @@
     <xacro:macro name="heron_hydro_model" params="namespace">
       <!-- List of hydrodynamic models this robot's links -->
-      <link name="${namespace}/base_link">
+      <link name="${namespace}base_link">
               <volume>${heron_volume}</volume>
               <box>

File: heron_description/urdf/heron.urdf.xacro (robot description, xacro)
@@ -27,10 +27,11 @@
 <robot name="heron" xmlns:xacro="http://www.ros.org/wiki/xacro" >
   <xacro:arg name="debug" default="0"/>
-  <xacro:arg name="namespace" default="/"/>
+  <xacro:arg name="namespace" default=""/>
+  <xacro:arg name="suffix_ns" default="$(arg namespace)"/>
   <!-- Include the ROV macro file -->
   <xacro:include filename="$(find heron_description)/urdf/base.xacro"/>
   <xacro:include filename="$(find heron_description)/urdf/gazebo.xacro"/>
   <!-- Create the heron -->
-  <xacro:heron_base namespace="$(arg namespace)">
+  <xacro:heron_base namespace="$(arg suffix_ns)">
     <!-- The underwater object plugin is given as an input block parameter to
      allow the addition of external models of manipulator units -->
@@ -41,5 +42,5 @@
         <debug>$(arg debug)</debug>
         <!-- Adding the hydrodynamic and hydrostatic parameters for the vehicle-->
-        <xacro:heron_hydro_model namespace="$(arg namespace)" />
+        <xacro:heron_hydro_model namespace="$(arg suffix_ns)" />
         <!--
           In case other modules are added to the vehicle (such as a manipulator)
@@ -55,5 +56,5 @@
   <gazebo>
     <plugin name="joint_state_publisher" filename="libjoint_state_publisher.so">
-      <robotNamespace>$(arg namespace)</robotNamespace>
+      <robotNamespace>/$(arg namespace)</robotNamespace>
       <updateRate>10</updateRate>
     </plugin>

File: heron_description/urdf/sensors.xacro (robot description, xacro)
@@ -5,9 +5,9 @@
     <plugin name="gps_controller" filename="libhector_gazebo_ros_gps.so">
       <updateRate>40</updateRate>
-      <robotNamespace>$(arg namespace)</robotNamespace>
-      <frameId>$(arg namespace)/navsat_link</frameId>
-      <bodyName>$(arg namespace)/navsat_link</bodyName>
-      <topicName>/$(arg namespace)/navsat/fix</topicName>
-      <velocityTopicName>/$(arg namespace)/navsat/velocity</velocityTopicName>
+      <robotNamespace>/$(arg namespace)</robotNamespace>
+      <frameId>$(arg suffix_ns)navsat_link</frameId>
+      <bodyName>$(arg suffix_ns)navsat_link</bodyName>
+      <topicName>/$(arg suffix_ns)navsat/fix</topicName>
+      <velocityTopicName>/$(arg suffix_ns)navsat/velocity</velocityTopicName>
       <referenceLatitude>49.9</referenceLatitude>
       <referenceLongitude>8.9</referenceLongitude>
@@ -17,8 +17,8 @@
     </plugin>
   </gazebo>
-  <link name="$(arg namespace)/navsat_link" />
+  <link name="$(arg suffix_ns)navsat_link" />
   <joint name="navsat_joint" type="fixed">
-    <parent link="$(arg namespace)/base_link" />
-    <child link="$(arg namespace)/navsat_link" />
+    <parent link="$(arg suffix_ns)base_link" />
+    <child link="$(arg suffix_ns)navsat_link" />
     <origin xyz="$(optenv HERON_NAVSAT_UBLOX_XYZ 0.015 0.050 0.072)"
       rpy="$(optenv HERON_NAVSAT_UBLOX_RPY 0.0 0.0 0.0)" />
@@ -27,9 +27,9 @@
     <gazebo>
       <plugin name="imu_controller" filename="libhector_gazebo_ros_imu.so">
-        <robotNamespace>$(arg namespace)</robotNamespace>
+        <robotNamespace>/$(arg namespace)</robotNamespace>
         <updateRate>50.0</updateRate>
-        <bodyName>$(arg namespace)/imu_link</bodyName>
-        <frameId>$(arg namespace)/imu_link</frameId>
-        <topicName>/$(arg namespace)/imu/data_raw</topicName>
+        <bodyName>$(arg suffix_ns)imu_link</bodyName>
+        <frameId>$(arg suffix_ns)imu_link</frameId>
+        <topicName>/$(arg suffix_ns)imu/data_raw</topicName>
         <accelDrift>0.005 0.005 0.005</accelDrift>
         <accelGaussianNoise>0.005 0.005 0.005</accelGaussianNoise>
@@ -40,9 +40,9 @@
       </plugin>
     </gazebo>
-    <link name="$(arg namespace)/imu_link" />
-    <joint name="$(arg namespace)/imu_joint" type="fixed">
+    <link name="$(arg suffix_ns)imu_link" />
+    <joint name="$(arg suffix_ns)imu_joint" type="fixed">
       <origin xyz="$(optenv HERON_IMU_UM6_XYZ -0.1397 0.0 0)" rpy="$(optenv HERON_IMU_UM6_RPY 0 0.0 0.0)" />
-      <parent link="$(arg namespace)/base_link" />
-      <child link="$(arg namespace)/imu_link" />
+      <parent link="$(arg suffix_ns)base_link" />
+      <child link="$(arg suffix_ns)imu_link" />
     </joint>
     <!-- Magnetometer -->
@@ -50,8 +50,8 @@
       <plugin name="mag_controller" filename="libhector_gazebo_ros_magnetic.so">
         <updateRate>50</updateRate>
-        <robotNamespace>$(arg namespace)</robotNamespace>
-        <bodyName>$(arg namespace)/imu_link</bodyName>
-        <frameId>$(arg namespace)/imu_link</frameId>
-        <topicName>/$(arg namespace)/imu/mag</topicName>
+        <robotNamespace>/$(arg namespace)</robotNamespace>
+        <bodyName>$(arg suffix_ns)imu_link</bodyName>
+        <frameId>$(arg suffix_ns)imu_link</frameId>
+        <topicName>/$(arg suffix_ns)imu/mag</topicName>
         <referenceHeading>90</referenceHeading>
         <drift>0.0005 0.0005 0.0005</drift>
@@ -63,7 +63,7 @@
       <plugin filename="libgazebo_ros_p3d.so" name="groundtruth_sim">
         <updateRate>20.0</updateRate>
-        <robotNamespace>$(arg namespace)</robotNamespace>
-        <bodyName>$(arg namespace)/base_link</bodyName>
-        <topicName>/$(arg namespace)/pose_gt</topicName>
+        <robotNamespace>/$(arg namespace)</robotNamespace>
+        <bodyName>$(arg suffix_ns)base_link</bodyName>
+        <topicName>/$(arg suffix_ns)pose_gt</topicName>
         <gaussianNoise>0.0</gaussianNoise>
         <frameName>world</frameName>

File: heron_description/urdf/snippets.xacro (robot description, xacro)
@@ -10,5 +10,5 @@
     be initialized in the actuators.xacro file.
   -->
-  <xacro:macro name="thruster_macro" params="robot_namespace thruster_id *origin">
+  <xacro:macro name="thruster_macro" params="robot_namespace suffix_ns thruster_id *origin">
     <!--
     Dummy link as place holder for the thruster frame,
@@ -16,5 +16,5 @@
     of the vehicle and may cause internal collisions if set otherwise
     -->
-    <link name="${robot_namespace}/thruster_${thruster_id}">
+    <link name="${suffix_ns}thruster_${thruster_id}">
       <visual>
         <geometry>
@@ -31,17 +31,17 @@
     </link>
     <!-- Joint between thruster link and vehicle base link -->
-    <joint name="${robot_namespace}/thruster_${thruster_id}_joint" type="continuous">
+    <joint name="${suffix_ns}thruster_${thruster_id}_joint" type="continuous">
       <xacro:insert_block name="origin" />
       <axis xyz="1 0 0" />
-      <parent link="${robot_namespace}/base_link" />
-      <child link="${robot_namespace}/thruster_${thruster_id}" />
+      <parent link="${suffix_ns}base_link" />
+      <child link="${suffix_ns}thruster_${thruster_id}" />
     </joint>
     <gazebo>
       <!-- Thruster ROS plugin -->
-      <plugin name="${robot_namespace}_${thruster_id}_thruster_model" filename="libthruster_ros_plugin.so">
+      <plugin name="${robot_namespace}thruster_${thruster_id}_thruster_model" filename="libthruster_ros_plugin.so">
         <!-- Name of the thruster link -->
-        <linkName>${robot_namespace}/thruster_${thruster_id}</linkName>
+        <linkName>${suffix_ns}thruster_${thruster_id}</linkName>
         <!-- Name of the joint between thruster and vehicle base link -->
-        <jointName>${robot_namespace}/thruster_${thruster_id}_joint</jointName>
+        <jointName>${suffix_ns}thruster_${thruster_id}_joint</jointName>
         <!-- Make the thruster aware of its id -->
         <thrusterID>${thruster_id}</thrusterID>
@@ -85,5 +85,5 @@
       </plugin>
     </gazebo>
-    <gazebo reference="${robot_namespace}/thruster_${thruster_id}">
+    <gazebo reference="${suffix_ns}thruster_${thruster_id}">
       <selfCollide>false</selfCollide>
     </gazebo>

Commit message: Fixed Heron accessories glitch with custom namespaces

File: heron_description/urdf/accessories.urdf.xacro (robot description, xacro)
@@ -9,6 +9,6 @@
     heron_base/launch/base.launch
   -->
-  <xacro:macro name="rear_plate" params="type namespace">
-    <link name="${namespace}rear_plate">
+  <xacro:macro name="rear_plate" params="type suffix_ns">
+    <link name="${suffix_ns}rear_plate">
       <visual>
         <origin xyz="0 0 0" rpy="0 0 0" />
@@ -20,9 +20,9 @@
     </link>
     <joint name="rear_plate_joint" type="fixed">
-      <parent link="${namespace}base_link" />
-      <child link="${namespace}rear_plate" />
+      <parent link="${suffix_ns}base_link" />
+      <child link="${suffix_ns}rear_plate" />
       <origin xyz="-0.1915 0.0 0.001" />
     </joint>
-    <gazebo reference="${namespace}rear_plate">
+    <gazebo reference="${suffix_ns}rear_plate">
       <material>Gazebo/DarkGrey</material>
     </gazebo>
@@ -31,5 +31,5 @@
   <xacro:include filename="accessories/novatel_smart6.urdf.xacro" />
   <xacro:if value="$(optenv HERON_NAVSAT_SMART6 0)">
-    <novatel_smart6 prefix="$(optenv HERON_NAVSAT_SMART6_MOUNT rear)" namespace="$(arg namespace)"/>
+    <novatel_smart6 prefix="$(optenv HERON_NAVSAT_SMART6_MOUNT rear)" suffix_ns="$(arg suffix_ns)"/>
     <joint name="$(optenv HERON_NAVSAT_SMART6_MOUNT rear)_navsat_joint" type="fixed">
     <origin xyz="$(optenv HERON_NAVSAT_SMART6_OFFSET -0.25 0 0.08)"
@@ -44,6 +44,6 @@
     <sick_lms1xx_mount prefix="$(optenv HERON_LASER_MOUNT front)"
                        topic="$(optenv HERON_LASER_TOPIC front/scan)"
-                       namespace="$(arg namespace)"/>
-    <rear_plate type="lidar" namespace="$(arg namespace)" />
+                       suffix_ns="$(arg suffix_ns)"/>
+    <rear_plate type="lidar" suffix_ns="$(arg suffix_ns)" />
     <joint name="$(optenv HERON_LASER_MOUNT front)_laser_mount_joint" type="fixed">
       <origin xyz="$(optenv HERON_LASER_OFFSET 0.0575 0 0.0115)"
@@ -56,5 +56,5 @@
   <xacro:include filename="accessories/axis_ptz.urdf.xacro" />
   <xacro:if value="$(optenv HERON_AXIS_PTZ 0)">
-    <axis_ptz prefix="$(optenv HERON_AXIS_PTZ_MOUNT axis_ptz)" namespace="$(arg namespace)"/>
+    <axis_ptz prefix="$(optenv HERON_AXIS_PTZ_MOUNT axis_ptz)" suffix_ns="$(arg suffix_ns)"/>
     <joint name="$(optenv HERON_AXIS_PTZ_MOUNT axis_ptz)_camera_joint" type="fixed">
     <origin xyz="$(optenv HERON_AXIS_PTZ_OFFSET -0.124 0 0.078)"
@@ -74,5 +74,5 @@
   </xacro:if>
   <xacro:unless value="$(optenv HERON_LASER 0)">
-    <rear_plate type="plain" namespace="$(arg suffix_ns)" />
+    <rear_plate type="plain" suffix_ns="$(arg suffix_ns)" />
   </xacro:unless>
 </robot>

File: heron_description/urdf/accessories/axis_ptz.urdf.xacro (robot description, xacro)
@@ -1,6 +1,6 @@
 <?xml version="1.0"?>
 <robot xmlns:xacro="http://www.ros.org/wiki/xacro">
-  <xacro:macro name="axis_ptz" params="prefix namespace">
-  <link name="${namespace}/${prefix}_camera_link">
+  <xacro:macro name="axis_ptz" params="prefix suffix_ns">
+  <link name="${suffix_ns}${prefix}_camera_link">
     <visual>
       <origin xyz="0 0 0" rpy="0 0 0" />

File: heron_description/urdf/accessories/novatel_smart6.urdf.xacro (robot description, xacro)
@@ -1,6 +1,6 @@
 <?xml version="1.0"?>
 <robot xmlns:xacro="http://www.ros.org/wiki/xacro">
-  <xacro:macro name="novatel_smart6" params="prefix namespace">
-  <link name="${namespace}/${prefix}_navsat">
+  <xacro:macro name="novatel_smart6" params="prefix suffix_ns">
+  <link name="${suffix_ns}${prefix}_navsat">
     <visual>
       <origin xyz="0 0 0" rpy="0 0 0" />

File: heron_description/urdf/accessories/sick_lms1xx_mount.urdf.xacro (robot description, xacro)
@@ -2,14 +2,14 @@
 <robot xmlns:xacro="http://www.ros.org/wiki/xacro">
   <xacro:include filename="$(find lms1xx)/urdf/sick_lms1xx.urdf.xacro" />
-  <xacro:macro name="sick_lms1xx_mount" params="prefix topic namespace">
-    <sick_lms1xx frame="${namespace}/${prefix}_laser" topic="${namespace}/${topic}" />
-    <link name="${namespace}/${prefix}_laser_mount"/>
-    <joint name="$${namespace}/{prefix}_laser_joint" type="fixed">
+  <xacro:macro name="sick_lms1xx_mount" params="prefix topic suffix_ns">
+    <sick_lms1xx frame="${suffix_ns}${prefix}_laser" topic="${suffix_ns}${topic}" />
+    <link name="${suffix_ns}${prefix}_laser_mount"/>
+    <joint name="${suffix_ns}${prefix}_laser_joint" type="fixed">
       <!-- This offset is from the base of the bracket to the LIDAR's focal point. -->
       <origin xyz="0 0 0.149" rpy="0 0 0" />
-      <parent link="${namespace}/${prefix}_laser_mount" />
-      <child link="${namespace}/${prefix}_laser" />
+      <parent link="${suffix_ns}${prefix}_laser_mount" />
+      <child link="${suffix_ns}${prefix}_laser" />
     </joint>
-    <gazebo reference="${namespace}/${prefix}_laser_mount">
+    <gazebo reference="${suffix_ns}${prefix}_laser_mount">
       <material>Gazebo/DarkGrey</material>
     </gazebo>
