Commit message: Further implementing namespaces

File: heron_description/urdf/base.xacro (robot description, xacro)
@@ -74,5 +74,5 @@
       </link>
       <!-- Dummy Link to contain the inertial information for base_link -->
-      <link name="dummy_link">
+      <link name="${namespace}/dummy_link">
         <inertial>
           <mass value="${mass}" />
@@ -86,5 +86,5 @@
       <joint name="dummy_to_base" type="fixed">
         <parent link="${namespace}/base_link" />
-        <child link="dummy_link" />
+        <child link="${namespace}/dummy_link" />
       </joint>
     <gazebo reference="${namespace}/base_link">

Commit message: Added simpler collision mesh

File: heron_description/urdf/base.xacro (robot description, xacro)
@@ -21,5 +21,5 @@
   this geometry as simple as possible to improve the performance the physics engine
   regarding the computation of collision forces) -->
-  <xacro:property name="collision_mesh_file" value="file://$(find heron_description)/meshes/heron_base.stl"/>
+  <xacro:property name="collision_mesh_file" value="file://$(find heron_description)/meshes/heron_collision.stl"/>
   <material name="gray"><color rgba="0.7 0.7 0.7 1.0"/></material>
   <material name="dark_gray"><color rgba="0.2 0.2 0.2 1.0"/></material>

Commit message: Changed mesh declarations to use packages instead of xacro finds

File: heron_description/urdf/base.xacro (robot description, xacro)
@@ -11,15 +11,4 @@
   <!-- Loading vehicle's specific macros -->
   <xacro:include filename="$(find heron_description)/urdf/snippets.xacro"/>
-  <!--
-    Visual mesh file for the vehicle, usually in DAE (Collada) format. Be sure to store the
-    mesh with the origin of the mesh on the same position of the center of mass, otherwise
-    the mesh pose will have to be corrected below in the <visual> block.
-    Open the meshes for the RexROV vehicle in Blender to see an example on the mesh placement.
-  -->
-  <xacro:property name="visual_mesh_file" value="file://$(find heron_description)/meshes/heron_base.stl"/>
-  <!-- Collision geometry mesh, usually in STL format (it is recommended to keep
-  this geometry as simple as possible to improve the performance the physics engine
-  regarding the computation of collision forces) -->
-  <xacro:property name="collision_mesh_file" value="file://$(find heron_description)/meshes/heron_collision.stl"/>
   <material name="gray"><color rgba="0.7 0.7 0.7 1.0"/></material>
   <material name="dark_gray"><color rgba="0.2 0.2 0.2 1.0"/></material>
@@ -42,5 +31,5 @@
           <origin xyz="0 0 0" rpy="0 0 0" />
           <geometry>
-            <mesh filename="file://$(find heron_description)/meshes/${side}_panel.stl" />
+            <mesh filename="package://heron_description/meshes/${side}_panel.stl" />
           </geometry>
           <material name="yellow" />
@@ -62,5 +51,5 @@
           <origin xyz="0 0 0" rpy="0 0 0"/>
           <geometry>
-            <mesh filename="${visual_mesh_file}" scale="1 1 1" />
+            <mesh filename="package://heron_description/meshes/heron_base.stl" scale="1 1 1" />
           </geometry>
           <material name="dark_gray" />
@@ -69,5 +58,5 @@
           <origin xyz="0 0 0" rpy="0 0 0"/>
           <geometry>
-            <mesh filename="${collision_mesh_file}" scale="1 1 1" />
+            <mesh filename="package://heron_description/meshes/heron_collision.stl" scale="1 1 1" />
           </geometry>
         </collision>

File: heron_description/urdf/snippets.xacro (robot description, xacro)
@@ -2,8 +2,4 @@
 <robot xmlns:xacro="http://www.ros.org/wiki/xacro">
   <!-- MACRO FOR THRUSTER UNITS  -->
-  <!-- Provide the propeller mesh in a separate file with the rotation axis
-  over propeller's frame X-axis in DAE (Collada) or STL format.
-  -->
-  <xacro:property name="prop_mesh_file" value="file://$(find heron_description)/meshes/prop.dae"/>
   <!--
     Thruster macro with integration of joint and link. The thrusters should
@@ -19,5 +15,5 @@
       <visual>
         <geometry>
-          <mesh filename="${prop_mesh_file}" scale="1 1 1" />
+          <mesh filename="package://heron_description/meshes/prop.dae" scale="1 1 1" />
         </geometry>
       </visual>

Commit message: Use a fixed joint for the thrusters unless we're in simulation; these joints are purely decorative outside gazebo, and the tf is not published except in simulation anyway

File: heron_description/urdf/base.xacro (robot description, xacro)
@@ -85,5 +85,14 @@
     <xacro:insert_block name="gazebo"/>
     <!-- Include the thruster modules -->
-    <xacro:include filename="$(find heron_description)/urdf/actuators.xacro"/>
+    <xacro:thruster_macro robot_namespace="$(arg namespace)" suffix_ns="$(arg suffix_ns)" thruster_id="0"
+      simulation="$(arg simulation)">
+      <!-- Right Thruster -->
+      <origin xyz="-0.53 -0.377654 -0.16" rpy="0 0 0" />
+    </xacro:thruster_macro>
+    <xacro:thruster_macro robot_namespace="$(arg namespace)" suffix_ns="$(arg suffix_ns)" thruster_id="1"
+      simulation="$(arg simulation)">
+      <!-- Left Thruster -->
+      <origin xyz="-0.53 0.377654 -0.16" rpy="0 0 0" />
+    </xacro:thruster_macro>s
     <!-- Include the sensor modules -->
     <xacro:include filename="$(find heron_description)/urdf/sensors.xacro"/>

File: heron_description/urdf/snippets.xacro (robot description, xacro)
@@ -6,5 +6,5 @@
     be initialized in the actuators.xacro file.
   -->
-  <xacro:macro name="thruster_macro" params="robot_namespace suffix_ns thruster_id *origin">
+  <xacro:macro name="thruster_macro" params="robot_namespace suffix_ns thruster_id *origin simulation:=false">
     <!--
     Dummy link as place holder for the thruster frame,
@@ -26,62 +26,72 @@
       </inertial>
     </link>
-    <!-- Joint between thruster link and vehicle base link -->
-    <joint name="${suffix_ns}thruster_${thruster_id}_joint" type="continuous">
-      <xacro:insert_block name="origin" />
-      <axis xyz="1 0 0" />
-      <parent link="${suffix_ns}base_link" />
-      <child link="${suffix_ns}thruster_${thruster_id}" />
-    </joint>
-    <gazebo>
-      <!-- Thruster ROS plugin -->
-      <plugin name="${robot_namespace}thruster_${thruster_id}_thruster_model" filename="libuuv_thruster_ros_plugin.so">
-        <!-- Name of the thruster link -->
-        <linkName>${suffix_ns}thruster_${thruster_id}</linkName>
-        <!-- Name of the joint between thruster and vehicle base link -->
-        <jointName>${suffix_ns}thruster_${thruster_id}_joint</jointName>
-        <!-- Make the thruster aware of its id -->
-        <thrusterID>${thruster_id}</thrusterID>
-        <!-- Gain of the input command signal -->
-        <gain>1</gain>
-        <!-- Maximum allowed input value for the input signal for thruster unit -->
-        <clampMax>100</clampMax>
-        <!-- Minimum allowed value for the input signal for thruster unit -->
-        <clampMin>-100</clampMin>
-        <!-- Minimum and maximum thrust force output allowed -->
-        <thrustMin>-35</thrustMin>
-        <thrustMax>35</thrustMax>
-        <!--
-        Value from 0 to 1 to set the efficiency of the output thrust force
-        Default value is 1.0
-        -->
-        <thrust_efficiency>1</thrust_efficiency>
-        <!--
-        Value from 0 to 1 to set the efficiency of the propeller as a factor
-        to be multiplied to the current value of the state variable at each
-        iteration.
-        Default value is 1.0
-        -->
-        <propeller_efficiency>1</propeller_efficiency>
-        <!-- 2) First order model -->
-        <dynamics>
-          <type>FirstOrder</type>
-          <timeConstant>0.05</timeConstant>
-        </dynamics>
-        <!-- 3) Linear interpolation
-        If you have access to the thruster's data sheet, for example,
-        you can enter samples of the curve's input and output values
-        and the thruster output will be found through linear interpolation
-        of the given samples.
-        -->
-        <conversion>
-          <type>LinearInterp</type>
-          <inputValues>-1.0 -0.8 -0.6 -0.4 -0.2 0 0.2 0.4 0.6 0.8 1.0</inputValues>
-          <outputValues>-19.88 -16.52 -12.6 -5.6 -1.4 0.0 2.24 9.52 21.28 28.0 33.6</outputValues>
-        </conversion>
-      </plugin>
-    </gazebo>
-    <gazebo reference="${suffix_ns}thruster_${thruster_id}">
-      <selfCollide>false</selfCollide>
-    </gazebo>
+    <xacro:if value="${simulation}">
+      <!-- Joint between thruster link and vehicle base link -->
+      <joint name="${suffix_ns}thruster_${thruster_id}_joint" type="continuous">
+        <xacro:insert_block name="origin" />
+        <axis xyz="1 0 0" />
+        <parent link="${suffix_ns}base_link" />
+        <child link="${suffix_ns}thruster_${thruster_id}" />
+      </joint>
+      <gazebo>
+        <!-- Thruster ROS plugin -->
+        <plugin name="${robot_namespace}thruster_${thruster_id}_thruster_model" filename="libuuv_thruster_ros_plugin.so">
+          <!-- Name of the thruster link -->
+          <linkName>${suffix_ns}thruster_${thruster_id}</linkName>
+          <!-- Name of the joint between thruster and vehicle base link -->
+          <jointName>${suffix_ns}thruster_${thruster_id}_joint</jointName>
+          <!-- Make the thruster aware of its id -->
+          <thrusterID>${thruster_id}</thrusterID>
+          <!-- Gain of the input command signal -->
+          <gain>1</gain>
+          <!-- Maximum allowed input value for the input signal for thruster unit -->
+          <clampMax>100</clampMax>
+          <!-- Minimum allowed value for the input signal for thruster unit -->
+          <clampMin>-100</clampMin>
+          <!-- Minimum and maximum thrust force output allowed -->
+          <thrustMin>-35</thrustMin>
+          <thrustMax>35</thrustMax>
+          <!--
+          Value from 0 to 1 to set the efficiency of the output thrust force
+          Default value is 1.0
+          -->
+          <thrust_efficiency>1</thrust_efficiency>
+          <!--
+          Value from 0 to 1 to set the efficiency of the propeller as a factor
+          to be multiplied to the current value of the state variable at each
+          iteration.
+          Default value is 1.0
+          -->
+          <propeller_efficiency>1</propeller_efficiency>
+          <!-- 2) First order model -->
+          <dynamics>
+            <type>FirstOrder</type>
+            <timeConstant>0.05</timeConstant>
+          </dynamics>
+          <!-- 3) Linear interpolation
+          If you have access to the thruster's data sheet, for example,
+          you can enter samples of the curve's input and output values
+          and the thruster output will be found through linear interpolation
+          of the given samples.
+          -->
+          <conversion>
+            <type>LinearInterp</type>
+            <inputValues>-1.0 -0.8 -0.6 -0.4 -0.2 0 0.2 0.4 0.6 0.8 1.0</inputValues>
+            <outputValues>-19.88 -16.52 -12.6 -5.6 -1.4 0.0 2.24 9.52 21.28 28.0 33.6</outputValues>
+          </conversion>
+        </plugin>
+      </gazebo>
+      <gazebo reference="${suffix_ns}thruster_${thruster_id}">
+        <selfCollide>false</selfCollide>
+      </gazebo>
+    </xacro:if>
+    <xacro:unless value="${simulation}">
+      <!-- On the real robot this joint is purely decorative; it's only used to produce thrust in gazebo -->
+      <joint name="${suffix_ns}thruster_${thruster_id}_joint" type="fixed">
+        <xacro:insert_block name="origin" />
+        <parent link="${suffix_ns}base_link" />
+        <child link="${suffix_ns}thruster_${thruster_id}" />
+      </joint>
+    </xacro:unless>
   </xacro:macro>
 </robot>
