Commit message: Switched UUV Sensor plugins to Gazebo plugins

File: heron_description/urdf/sensors.xacro (robot description, xacro)
@@ -1,24 +1,5 @@
 <?xml version="1.0"?>
 <robot xmlns:xacro="http://www.ros.org/wiki/xacro">
-  <!--
-    Some examples of sensors that can be added to the vehicle frame.
-    Set the origin of the sensor frames correctly for your application
-    Look into the sensor macros in the package uuv_sensor_ros_plugins/urdf for
-    more examples or add you own custom sensor units.
-  -->
   <!-- GPS -->
-  <!-- <xacro:gps_sensor_macro
-    namespace="${namespace}"
-    parent_link="${namespace}/base_link"
-    gps_topic="navsat/fix"
-    update_rate="30"
-    mass_gps_sensor="0.001"
-    horizontal_pos_std_dev="0.01"
-    vertical_pos_std_dev="0.01"
-    horizontal_vel_std_dev="0.01"
-    vertical_vel_std_dev="0.01">
-    <inertia ixx="0.00001" ixy="0.0" ixz="0.0" iyy="0.00001" iyz="0.0" izz="0.00001" />
-    <origin xyz="0 0 0" rpy="0 0 0" />
-  </xacro:gps_sensor_macro> -->
   <gazebo>
     <plugin name="gps_controller" filename="libhector_gazebo_ros_gps.so">
@@ -37,64 +18,41 @@
   </gazebo>
   <!-- IMU -->
-  <!-- <xacro:imu_plugin_macro
-      namespace="${namespace}"
-      imu_suffix=""
-      parent_link="${namespace}/base_link"
-      imu_topic="imu/data_raw"
-      mass_imu_sensor="0.015"
-      gyroscope_noise_density="0.0003394"
-      gyroscope_random_walk="0.000038785"
-      gyroscope_bias_correlation_time="1000.0"
-      gyroscope_turn_on_bias_sigma="0.0087"
-      accelerometer_noise_density="0.004"
-      accelerometer_random_walk="0.006"
-      accelerometer_bias_correlation_time="300.0"
-      accelerometer_turn_on_bias_sigma="0.1960"
-      orientation_noise="0.01"
-      enable_local_ned_frame="false"
-      reference_frame="world"
-      update_rate="50">
-      <inertia ixx="0.00001" ixy="0.0" ixz="0.0" iyy="0.00001" iyz="0.0" izz="0.00001" />
-      <origin xyz="0 0 0" rpy="0 0 0" />
-    </xacro:imu_plugin_macro> -->
-    <xacro:imu_plugin_macro
-        namespace="${namespace}"
-        imu_suffix=""
-        parent_link="${namespace}/base_link"
-        imu_topic="imu/data_raw"
-        mass_imu_sensor="0.015"
-        gyroscope_noise_density="0.0003394"
-        gyroscope_random_walk="0.000038785"
-        gyroscope_bias_correlation_time="1000.0"
-        gyroscope_turn_on_bias_sigma="0.0087"
-        accelerometer_noise_density="0.04"
-        accelerometer_random_walk="0.006"
-        accelerometer_bias_correlation_time="300.0"
-        accelerometer_turn_on_bias_sigma="0.1960"
-        orientation_noise="0.01"
-        enable_local_ned_frame="false"
-        reference_frame="world"
-        update_rate="50">
-        <inertia ixx="0.00001" ixy="0.0" ixz="0.0" iyy="0.00001" iyz="0.0" izz="0.00001" />
-        <origin xyz="0 0 0" rpy="0 0 0" />
-      </xacro:imu_plugin_macro>
-    <xacro:magnetometer_plugin_macro
-        namespace="${namespace}"
-        suffix=""
-        parent_link="${namespace}/base_link"
-        topic="imu/mag_sim"
-        mass="0.015"
-        update_rate="50"
-        mag_intensity="65.0"
-        noise_xy="0.25"
-        noise_z="0.35"
-        turn_on_bias="2.0">
-        <inertia ixx="0.00001" ixy="0.0" ixz="0.0" iyy="0.00001" iyz="0.0" izz="0.00001" />
-        <origin xyz="0 0 0" rpy="0 0 0" />
-      </xacro:magnetometer_plugin_macro>
-      <!-- Mount a Perfect Pose 3D sensor. -->
-      <xacro:default_pose_3d_macro
-        namespace="${namespace}"
-        parent_link="${namespace}/base_link"
-        inertial_reference_frame="world" />
+  <gazebo>
+   <plugin name="imu_controller" filename="libhector_gazebo_ros_imu.so">
+     <robotNamespace>$(arg namespace)</robotNamespace>
+     <updateRate>50.0</updateRate>
+     <bodyName>imu_link</bodyName>
+     <topicName>imu/data</topicName>
+     <accelDrift>0.005 0.005 0.005</accelDrift>
+     <accelGaussianNoise>0.005 0.005 0.005</accelGaussianNoise>
+     <rateDrift>0.005 0.005 0.005 </rateDrift>
+     <rateGaussianNoise>0.005 0.005 0.005 </rateGaussianNoise>
+     <headingDrift>0.005</headingDrift>
+     <headingGaussianNoise>0.005</headingGaussianNoise>
+   </plugin>
+ </gazebo>
+ <!-- Magnetometer -->
+ <gazebo>
+   <plugin name="mag_controller" filename="libhector_gazebo_ros_magnetic.so">
+     <updateRate>50</updateRate>
+     <robotNamespace>$(arg namespace)</robotNamespace>
+     <bodyName>imu_link</bodyName>
+     <frameId>imu_link</frameId>
+     <topicName>/imu/mag</topicName>
+     <referenceHeading>90</referenceHeading>
+     <drift>0.0005 0.0005 0.0005</drift>
+     <gaussianNoise>0.025 0.025 0.025</gaussianNoise>
+   </plugin>
+ </gazebo>
+    <!-- Mount a Perfect Pose 3D sensor. -->
+    <gazebo>
+      <plugin filename="libgazebo_ros_p3d.so" name="quadrotor_groundtruth_sim">
+        <updateRate>20.0</updateRate>
+        <robotNamespace>$(arg namespace)</robotNamespace>
+        <bodyName>base_link</bodyName>
+        <topicName>pose_gt</topicName>
+        <gaussianNoise>0.0</gaussianNoise>
+        <frameName>world</frameName>
+      </plugin>
+    </gazebo>
 </robot>

Commit message: Additional updates so Gazebo sensor plugins would work with namespaces

File: heron_description/urdf/sensors.xacro (robot description, xacro)
@@ -22,6 +22,7 @@
      <robotNamespace>$(arg namespace)</robotNamespace>
      <updateRate>50.0</updateRate>
-     <bodyName>imu_link</bodyName>
-     <topicName>imu/data</topicName>
+     <bodyName>$(arg namespace)/imu_link</bodyName>
+     <frameId>$(arg namespace)/imu_link</frameId>
+     <topicName>/$(arg namespace)/imu/data_raw</topicName>
      <accelDrift>0.005 0.005 0.005</accelDrift>
      <accelGaussianNoise>0.005 0.005 0.005</accelGaussianNoise>
@@ -32,4 +33,10 @@
    </plugin>
  </gazebo>
+ <link name="$(arg namespace)/imu_link" />
+ <joint name="$(arg namespace)/imu_joint" type="fixed">
+  <origin xyz="-0.1397 0 0" rpy="0 0 0" />
+  <parent link="$(arg namespace)/base_link" />
+  <child link="$(arg namespace)/imu_link" />
+</joint>
  <!-- Magnetometer -->
  <gazebo>
@@ -37,7 +44,7 @@
      <updateRate>50</updateRate>
      <robotNamespace>$(arg namespace)</robotNamespace>
-     <bodyName>imu_link</bodyName>
-     <frameId>imu_link</frameId>
-     <topicName>/imu/mag</topicName>
+     <bodyName>$(arg namespace)/imu_link</bodyName>
+     <frameId>$(arg namespace)/imu_link</frameId>
+     <topicName>/$(arg namespace)/imu/mag</topicName>
      <referenceHeading>90</referenceHeading>
      <drift>0.0005 0.0005 0.0005</drift>
@@ -45,14 +52,14 @@
    </plugin>
  </gazebo>
-    <!-- Mount a Perfect Pose 3D sensor. -->
-    <gazebo>
-      <plugin filename="libgazebo_ros_p3d.so" name="quadrotor_groundtruth_sim">
-        <updateRate>20.0</updateRate>
-        <robotNamespace>$(arg namespace)</robotNamespace>
-        <bodyName>base_link</bodyName>
-        <topicName>pose_gt</topicName>
-        <gaussianNoise>0.0</gaussianNoise>
-        <frameName>world</frameName>
-      </plugin>
-    </gazebo>
+  <!-- Mount a Perfect Pose 3D sensor. -->
+  <gazebo>
+    <plugin filename="libgazebo_ros_p3d.so" name="groundtruth_sim">
+      <updateRate>20.0</updateRate>
+      <robotNamespace>$(arg namespace)</robotNamespace>
+      <bodyName>$(arg namespace)/base_link</bodyName>
+      <topicName>/$(arg namespace)/pose_gt</topicName>
+      <gaussianNoise>0.0</gaussianNoise>
+      <frameName>world</frameName>
+    </plugin>
+  </gazebo>
 </robot>

Commit message: Added envvars to change sensor locations and attached GPS info to separate sensor frame

File: heron_description/urdf/sensors.xacro (robot description, xacro)
@@ -6,6 +6,6 @@
       <updateRate>40</updateRate>
       <robotNamespace>$(arg namespace)</robotNamespace>
-      <frameId>$(arg namespace)/base_link</frameId>
-      <bodyName>$(arg namespace)/base_link</bodyName>
+      <frameId>$(arg namespace)/navsat_link</frameId>
+      <bodyName>$(arg namespace)/navsat_link</bodyName>
       <topicName>/$(arg namespace)/navsat/fix</topicName>
       <velocityTopicName>/$(arg namespace)/navsat/vel</velocityTopicName>
@@ -17,4 +17,11 @@
     </plugin>
   </gazebo>
+  <link name="$(arg namespace)/navsat_link" />
+  <joint name="navsat_joint" type="fixed">
+    <parent link="$(arg namespace)/base_link" />
+    <child link="$(arg namespace)/navsat_link" />
+    <origin xyz="$(optenv HERON_NAVSAT_UBLOX_XYZ 0.015 0.050 0.072)"
+              rpy="$(optenv HERON_NAVSAT_UBLOX_RPY 0.0 0.0 0.0)" />
+  </joint>
   <!-- IMU -->
   <gazebo>
@@ -35,5 +42,5 @@
  <link name="$(arg namespace)/imu_link" />
  <joint name="$(arg namespace)/imu_joint" type="fixed">
-  <origin xyz="-0.1397 0 0" rpy="0 0 0" />
+  <origin xyz="$(optenv HERON_IMU_UM6_XYZ -0.1397 0.0 0)" rpy="$(optenv HERON_IMU_UM6_RPY 0 0.0 0.0)" />
   <parent link="$(arg namespace)/base_link" />
   <child link="$(arg namespace)/imu_link" />

Commit message: Fixed spacing using Atom auto-indent

File: heron_description/urdf/sensors.xacro (robot description, xacro)
@@ -22,51 +22,51 @@
     <child link="$(arg namespace)/navsat_link" />
     <origin xyz="$(optenv HERON_NAVSAT_UBLOX_XYZ 0.015 0.050 0.072)"
-              rpy="$(optenv HERON_NAVSAT_UBLOX_RPY 0.0 0.0 0.0)" />
-  </joint>
-  <!-- IMU -->
-  <gazebo>
-   <plugin name="imu_controller" filename="libhector_gazebo_ros_imu.so">
-     <robotNamespace>$(arg namespace)</robotNamespace>
-     <updateRate>50.0</updateRate>
-     <bodyName>$(arg namespace)/imu_link</bodyName>
-     <frameId>$(arg namespace)/imu_link</frameId>
-     <topicName>/$(arg namespace)/imu/data_raw</topicName>
-     <accelDrift>0.005 0.005 0.005</accelDrift>
-     <accelGaussianNoise>0.005 0.005 0.005</accelGaussianNoise>
-     <rateDrift>0.005 0.005 0.005 </rateDrift>
-     <rateGaussianNoise>0.005 0.005 0.005 </rateGaussianNoise>
-     <headingDrift>0.005</headingDrift>
-     <headingGaussianNoise>0.005</headingGaussianNoise>
-   </plugin>
- </gazebo>
- <link name="$(arg namespace)/imu_link" />
- <joint name="$(arg namespace)/imu_joint" type="fixed">
-  <origin xyz="$(optenv HERON_IMU_UM6_XYZ -0.1397 0.0 0)" rpy="$(optenv HERON_IMU_UM6_RPY 0 0.0 0.0)" />
-  <parent link="$(arg namespace)/base_link" />
-  <child link="$(arg namespace)/imu_link" />
-</joint>
- <!-- Magnetometer -->
- <gazebo>
-   <plugin name="mag_controller" filename="libhector_gazebo_ros_magnetic.so">
-     <updateRate>50</updateRate>
-     <robotNamespace>$(arg namespace)</robotNamespace>
-     <bodyName>$(arg namespace)/imu_link</bodyName>
-     <frameId>$(arg namespace)/imu_link</frameId>
-     <topicName>/$(arg namespace)/imu/mag</topicName>
-     <referenceHeading>90</referenceHeading>
-     <drift>0.0005 0.0005 0.0005</drift>
-     <gaussianNoise>0.025 0.025 0.025</gaussianNoise>
-   </plugin>
- </gazebo>
-  <!-- Mount a Perfect Pose 3D sensor. -->
-  <gazebo>
-    <plugin filename="libgazebo_ros_p3d.so" name="groundtruth_sim">
-      <updateRate>20.0</updateRate>
-      <robotNamespace>$(arg namespace)</robotNamespace>
-      <bodyName>$(arg namespace)/base_link</bodyName>
-      <topicName>/$(arg namespace)/pose_gt</topicName>
-      <gaussianNoise>0.0</gaussianNoise>
-      <frameName>world</frameName>
-    </plugin>
-  </gazebo>
-</robot>
+      rpy="$(optenv HERON_NAVSAT_UBLOX_RPY 0.0 0.0 0.0)" />
+    </joint>
+    <!-- IMU -->
+    <gazebo>
+      <plugin name="imu_controller" filename="libhector_gazebo_ros_imu.so">
+        <robotNamespace>$(arg namespace)</robotNamespace>
+        <updateRate>50.0</updateRate>
+        <bodyName>$(arg namespace)/imu_link</bodyName>
+        <frameId>$(arg namespace)/imu_link</frameId>
+        <topicName>/$(arg namespace)/imu/data_raw</topicName>
+        <accelDrift>0.005 0.005 0.005</accelDrift>
+        <accelGaussianNoise>0.005 0.005 0.005</accelGaussianNoise>
+        <rateDrift>0.005 0.005 0.005 </rateDrift>
+        <rateGaussianNoise>0.005 0.005 0.005 </rateGaussianNoise>
+        <headingDrift>0.005</headingDrift>
+        <headingGaussianNoise>0.005</headingGaussianNoise>
+      </plugin>
+    </gazebo>
+    <link name="$(arg namespace)/imu_link" />
+    <joint name="$(arg namespace)/imu_joint" type="fixed">
+      <origin xyz="$(optenv HERON_IMU_UM6_XYZ -0.1397 0.0 0)" rpy="$(optenv HERON_IMU_UM6_RPY 0 0.0 0.0)" />
+      <parent link="$(arg namespace)/base_link" />
+      <child link="$(arg namespace)/imu_link" />
+    </joint>
+    <!-- Magnetometer -->
+    <gazebo>
+      <plugin name="mag_controller" filename="libhector_gazebo_ros_magnetic.so">
+        <updateRate>50</updateRate>
+        <robotNamespace>$(arg namespace)</robotNamespace>
+        <bodyName>$(arg namespace)/imu_link</bodyName>
+        <frameId>$(arg namespace)/imu_link</frameId>
+        <topicName>/$(arg namespace)/imu/mag</topicName>
+        <referenceHeading>90</referenceHeading>
+        <drift>0.0005 0.0005 0.0005</drift>
+        <gaussianNoise>0.025 0.025 0.025</gaussianNoise>
+      </plugin>
+    </gazebo>
+    <!-- Mount a Perfect Pose 3D sensor. -->
+    <gazebo>
+      <plugin filename="libgazebo_ros_p3d.so" name="groundtruth_sim">
+        <updateRate>20.0</updateRate>
+        <robotNamespace>$(arg namespace)</robotNamespace>
+        <bodyName>$(arg namespace)/base_link</bodyName>
+        <topicName>/$(arg namespace)/pose_gt</topicName>
+        <gaussianNoise>0.0</gaussianNoise>
+        <frameName>world</frameName>
+      </plugin>
+    </gazebo>
+  </robot>

Commit message: Rename the UM6 IMU env vars to remove the reference to UM6; make them generic IMU vars instead

File: heron_description/urdf/sensors.xacro (robot description, xacro)
@@ -42,5 +42,5 @@
     <link name="$(arg suffix_ns)imu_link" />
     <joint name="$(arg suffix_ns)imu_joint" type="fixed">
-      <origin xyz="$(optenv HERON_IMU_UM6_XYZ -0.1397 0.0 0)" rpy="$(optenv HERON_IMU_UM6_RPY 0 0.0 0.0)" />
+      <origin xyz="$(optenv HERON_IMU_XYZ -0.1397 0.0 0)" rpy="$(optenv HERON_IMU_RPY 0 0.0 0.0)" />
       <parent link="$(arg suffix_ns)base_link" />
       <child link="$(arg suffix_ns)imu_link" />

Commit message: Description now uses environment variable for reference latitude and longitude as in navsat transform.

File: heron_description/urdf/sensors.xacro (robot description, xacro)
@@ -3,4 +3,8 @@
   <!-- GPS -->
   <gazebo>
+    <xacro:property name="datum_env" value="$(optenv GPS_DATUM '49.9, 8.9')"/>
+    <xacro:property name="datum" value="${map(float, datum_env.split(','))}" />
+    <xacro:property name="datum_lat" value="${datum[0]}" />
+    <xacro:property name="datum_lon" value="${datum[1]}" />
     <plugin name="gps_controller" filename="libhector_gazebo_ros_gps.so">
       <updateRate>40</updateRate>
@@ -10,6 +14,6 @@
       <topicName>/$(arg suffix_ns)navsat/fix</topicName>
       <velocityTopicName>/$(arg suffix_ns)navsat/velocity</velocityTopicName>
-      <referenceLatitude>49.9</referenceLatitude>
-      <referenceLongitude>8.9</referenceLongitude>
+      <referenceLatitude>${datum_lat}</referenceLatitude>
+      <referenceLongitude>${datum_lon}</referenceLongitude>
       <referenceHeading>90</referenceHeading>
       <referenceAltitude>0</referenceAltitude>

Commit message: Compatibility change to sensors.xacro for noetic(python3).

File: heron_description/urdf/sensors.xacro (robot description, xacro)
@@ -4,5 +4,5 @@
   <gazebo>
     <xacro:property name="datum_env" value="$(optenv GPS_DATUM '49.9, 8.9')"/>
-    <xacro:property name="datum" value="${map(float, datum_env.split(','))}" />
+    <xacro:property name="datum" value="${list(map(float, datum_env.split(',')))}" />
     <xacro:property name="datum_lat" value="${datum[0]}" />
     <xacro:property name="datum_lon" value="${datum[1]}" />
